File: MY-MP3.kicad_pcb (KiCad board)
At the start: 4 copper layers, 13 x 1.4 mm, 75 parts, among them J1 microSD, J2 USB_C_Receptacle, J3 JST_2mm_LiPo, J4 Adafruit 5393 Headers, J5 Adafruit 5394 Headers, J6 Newxie Headers, J7 AudioJack3_SwitchTR, Q1 DMG3415U, SW1 SMD_6x3.5mm_h2.5mm, SW2 SMD_6x3.5mm_h2.5mm, U1 STM32L4R5VITx, U2 CODECODER-VS1053B_LQFP48_, U3 RT9080-3.3, U4 MAX17048, U6 MCP73831-2-OT, U7 AP7312-1833W6, Y1 ABM3-12.288MHZ-D2Y-T, Y2 8 mHz

Commit message: Finish Schematic and start PCB
Parts:
- removed J5: Adafruit 5394 Headers, Connector_PinSocket_2.54mm:PinSocket_1x11_P2.54mm_Vertical
- removed J6: Newxie Headers, Connector_PinSocket_2.54mm:PinSocket_1x07_P2.54mm_Vertical
- added C28: 470nF, PCM_SparkFun-Capacitor:C_0402_1005Metric, F.Cu at (142.5, 130.0)
- added C29: 1.0uF, PCM_SparkFun-Capacitor:C_0603_1608Metric, F.Cu at (149.8, 130.0)
- added C30: 0.1uF, PCM_SparkFun-Capacitor:C_0603_1608Metric, F.Cu at (142.0, 127.5)
- added C31: 0.1uF, PCM_SparkFun-Capacitor:C_0603_1608Metric, F.Cu at (147.5, 102.0)
- added J9: Conn_01x04_FPC, Connector_FFC-FPC:Amphenol_F32Q-1A7x1-11004_1x04-1MP_P0.5mm_Horizontal, B.Cu at (170.2, 122.0)
- added LED3: LED_0603_Red, PCM_LED_SMD_AKL:LED_0603_1608Metric, F.Cu at (174.5, 51.5)
- added SW3: BTN_POW, PCM_SparkFun-Switch:Push_SMD_RA_4.5x3.4mm, F.Cu at (143.5, 50.0)
- added SW4: BTN_VUP, PCM_SparkFun-Switch:Push_SMD_RA_4.5x3.4mm, F.Cu at (174.5, 64.5)
- added SW5: BTN_VDN, PCM_SparkFun-Switch:Push_SMD_RA_4.5x3.4mm, F.Cu at (174.5, 70.0)
- added SW6: Nav Switch, PCM_SparkFun-Switch:Navigation_SMD_9.9x9.9mm, B.Cu at (157.7, 121.8)
- added SW7: BTN_OPT, PCM_SparkFun-Switch:Push_SMD_6x3.5mm, B.Cu at (168.5, 114.0)
- added SW8: BTN_SEL, PCM_SparkFun-Switch:Push_SMD_6x3.5mm, B.Cu at (149.0, 114.0)
- added U5: STM6601, Package_DFN_QFN:TDFN-12_2x3mm_P0.5mm, F.Cu at (145.7, 128.8)
- C12, C17, C18, C19, C20, C21, J4: moved to B.Cu
- moved J4 103.7 mm to (169.5, 66.9), turned to 180 degrees
- moved R8 80.6 mm to (174.0, 59.0), turned to 90 degrees
- moved R25 77.5 mm to (165.5, 51.5), turned to -90 degrees
- moved R20 77.5 mm to (169.5, 51.5), turned to 90 degrees
- moved R16 75.5 mm to (173.8, 54.5)
- moved R3 75.2 mm to (172.5, 115.0)
- moved C3 75.1 mm to (162.0, 122.5)
- moved U6 69.9 mm to (157.5, 126.0)
- moved U3 68.2 mm to (153.5, 121.0)
- moved C6 67.7 mm to (158.0, 64.5), turned to 180 degrees
- moved C19 67.4 mm to (163.0, 110.0), turned to 180 degrees
- moved C2 66.9 mm to (149.3, 125.0), turned to 180 degrees
- moved R6 66.2 mm to (165.5, 70.0)
- moved C27 65.6 mm to (159.0, 117.5), turned to 90 degrees
- moved R13 65.5 mm to (149.5, 133.0), turned to 90 degrees
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Connections:
- R16 pad 1: Net-(D1-K) -> Net-(LED3-A)
- R16 pad 2: Net-(U3-EN) -> VBATT
- U1 pad 15: /TFT_DC -> /JOY_X
- U1 pad 16: /TFT_SD_CS -> /JOY_Y
- U1 pad 17: unconnected-(U1-PC2-Pad17) -> /TFT_DC
- U1 pad 18: unconnected-(U1-PC3-Pad18) -> /TFT_SD_CS
- U1 pad 38: unconnected-(U1-PE7-Pad38) -> /NPB_OUT
- U1 pad 39: unconnected-(U1-PE8-Pad39) -> /STM6601_NINT
- U1 pad 5: unconnected-(U1-PE6-Pad5) -> /NVCC_LO
- U1 pad 55: unconnected-(U1-PD8-Pad55) -> /BTN_OPT
- U1 pad 56: unconnected-(U1-PD9-Pad56) -> /BTN_SEL
- U1 pad 57: unconnected-(U1-PD10-Pad57) -> /BTN_PLAY
- U1 pad 58: unconnected-(U1-PD11-Pad58) -> /BTN_UP
- U1 pad 59: unconnected-(U1-PD12-Pad59) -> /BTN_DN
- U1 pad 6: 3.3V -> Net-(U1-VBAT)
- U1 pad 60: unconnected-(U1-PD13-Pad60) -> /BTN_TRACK
- U1 pad 61: unconnected-(U1-PD14-Pad61) -> /BTN_SEEK
- U1 pad 87: unconnected-(U1-PD6-Pad87) -> /BTN_VUP
- U1 pad 88: unconnected-(U1-PD7-Pad88) -> /BTN_VDN
- U3 pad 3: Net-(U3-EN) -> /LDO_EN
- U4 pad 3: 3.3V -> VBATT
Routing:
- added copper zone on In1.Cu, net 3.3V
- added copper zone on In2.Cu, net GND
Other:
- board size 13 x 1.4 mm -> 37 x 90 mm
- board text added: "LED1"

Commit message: Finish PCB
Parts:
- removed J9: Conn_01x04_FPC, Connector_FFC-FPC:Amphenol_F32Q-1A7x1-11004_1x04-1MP_P0.5mm_Horizontal
- C1, C10, C14, C16, C2, C22, C23, C25, C26, C27, C28, C29, C3, C30, C31, C7, C8, C9, D1, FB1, FB2, J2, J3, J7, Q1, R1, R10, R12, R13, R14, R15, R16, R18, R19, R2, R20, R22, R23, R25, R4, R5, R6, R7, R8, R9, U2, U3, U4, U5, U6, U7, Y1: moved to B.Cu
- J4: footprint Connector_PinSocket_2.54mm:PinSocket_1x11_P2.54mm_Vertical -> Connector_PinSocket_2.54mm:PinSocket_1x11_P2.54mm_Vertical_SMD_Pin1Left; moved to F.Cu
- SW6, SW7, SW8: moved to F.Cu
- moved R25 75.5 mm to (174.5, 126.5), turned to 90 degrees
- moved LED2 75.3 mm to (174.5, 126.5), turned to -90 degrees
- moved LED3 75.2 mm to (169.5, 126.5)
- moved R20 75.0 mm to (172.0, 126.5), turned to -90 degrees
- moved LED1 75.0 mm to (172.0, 126.5), turned to -90 degrees
- moved R16 72.1 mm to (169.5, 126.5), turned to -90 degrees
- moved R21 59.0 mm to (147.7, 60.0), turned to -90 degrees
- moved SW1 58.7 mm to (150.0, 64.0)
- moved SW2 58.6 mm to (150.0, 69.0)
- moved D3 55.1 mm to (150.7, 60.0), turned to 90 degrees
- moved C15 52.1 mm to (152.7, 60.0), turned to 90 degrees
- moved R3 45.7 mm to (153.2, 73.5), turned to 90 degrees
- moved D2 45.4 mm to (148.7, 73.5), turned to 90 degrees
- moved C24 42.3 mm to (150.7, 73.5), turned to 90 degrees
- moved SW4 42.1 mm to (146.5, 96.0), turned to 90 degrees
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Routing:
- net GND: track 0.00 -> 344.7 mm, vias 0 -> 24
- net 1.8V: track 0.00 -> 260.8 mm, vias 0 -> 8
- net GNDA: track 0.00 -> 254.5 mm, vias 0 -> 5
- net 3.3V: track 0.00 -> 192.6 mm, vias 0 -> 18
- net Net-(U5-~{PB}): track 0.00 -> 165.4 mm, vias 0 -> 3
- net /BTN_DN: track 0.00 -> 108.0 mm, vias 0 -> 8
- net /NRST: track 0.00 -> 104.6 mm, vias 0 -> 2
- net /BTN_SEEK: track 0.00 -> 96.8 mm, vias 0 -> 2
- net /BTN_UP: track 0.00 -> 90.7 mm, vias 0 -> 7
- net /BTN_PLAY: track 0.00 -> 90.1 mm, vias 0 -> 12
- net /BTN_OPT: track 0.00 -> 90.0 mm, vias 0 -> 7
- net /LED: track 0.00 -> 85.8 mm, vias 0 -> 3
- net VBATT: track 0.00 -> 82.5 mm, vias 0 -> 5
- net VBUS: track 0.00 -> 81.5 mm, vias 0 -> 1
- net 3.3V_A: track 0.00 -> 80.9 mm, vias 0 -> 11
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- added copper zone on In1.Cu, net 3.3V_A
- added copper zone on In1.Cu, net VBATT
Other:
- board size 37 x 90 mm -> 32.4 x 105.7 mm
- board text removed: "LED1"
